File: ATMega128_Breakout.sch (KiCad schematic (older format))
At the start: 21 parts, among them IC1 ATMEGA128-A, J2 SIL8, P1 CONN_10, P2 CONN_10, P3 CONN_10, P4 CONN_10, P5 CONN_01X01, P6 CONN_7, P8 CONN_5X2, SW1 rst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

Commit message: Updated Designs
Parts:
- removed C5: 0.1uF, ~, symbol C
- removed P6: CONN_7, symbol CONN_7
- added C6, C7, C8: 0.1uF, ~, symbol C
- added CON1: USB-MICRO-B, symbol USB-MICRO-B
- added P10, P6, P7, P9: CONN_01X01, symbol CONN_01X01
- added R5: R, symbol R
- added U1: CP2102, symbol CP2102
Connections:
- net +5V: now also P4.10 (P10), C6.1, CON1.1 (VBUS), U1.7 (REGIN), U1.8 (VBUS); no longer IC1.62 (AREF), P3.1 (P1)
- net GND: now also P4.9 (P9), C6.2, C7.1, CON1.4 (ID), CON1.5 (GND), U1.3 (GND); no longer P3.2 (P2)
- net RST: now also C8.2
- net RX0: now also P4.1 (P1), R5.1; no longer J2.1
- net SCL: now also P3.1 (P1); no longer P4.10 (P10)
- net SDA: now also P3.2 (P2); no longer P4.9 (P9)
- net TX0: now also P4.2 (P2), U1.25 (RXD); no longer J2.2
- net at J2.3: now also IC1.37 ((A10)PC2); no longer IC1.4 (PE2(XCK0/AIN0))
- net at J2.4: now also IC1.38 ((A11)PC3); no longer IC1.5 (PE3(OC3A/AIN1))
- net at J2.5: now also IC1.39 ((A12)PC4); no longer IC1.6 (PE4(OC3B/INT4))
- net at J2.6: now also IC1.40 ((A13)PC5); no longer IC1.7 (PE5(OC3C/INT5))
- net at J2.7: now also IC1.41 ((A14)PC6); no longer IC1.8 (PE6(T3/INT6))
- net at J2.8: now also IC1.42 ((A15)PC7); no longer IC1.9 (PE7(IC3/INT7))
- net at IC1.35 ((A8)PC0): now also J2.1; no longer P4.1 (P1)
- net at IC1.36 ((A9)PC1): now also J2.2; no longer P4.2 (P2)
- net at P4.3 (P3): now also IC1.4 (PE2(XCK0/AIN0)); no longer IC1.37 ((A10)PC2)
- net at P4.4 (P4): now also IC1.5 (PE3(OC3A/AIN1)); no longer IC1.38 ((A11)PC3)
- net at P4.5 (P5): now also IC1.6 (PE4(OC3B/INT4)); no longer IC1.39 ((A12)PC4)
- net at P4.6 (P6): now also IC1.7 (PE5(OC3C/INT5)); no longer IC1.40 ((A13)PC5)
- net at P4.7 (P7): now also IC1.8 (PE6(T3/INT6)); no longer IC1.41 ((A14)PC6)
- net at P4.8 (P8): now also IC1.9 (PE7(IC3/INT7)); no longer IC1.42 ((A15)PC7)
- net Aref: now reaches P2.1 (P1)
- net Aref: now also IC1.62 (AREF)
- new net: CON1.2 (D-), U1.5 (D-)
- new net: CON1.3 (D+), U1.4 (D+)
- new net: R5.2, U1.26 (TXD)
- new net: C8.1, U1.28 (DTR)
- new net: C7.2, U1.6 (VDD)
- no-connect marks 21 -> 44
Other:
- moved on the sheet: J2, P4, P5, P8

Commit message: Updated
Parts:
- added R4: 470r, symbol R
- R5: value R -> 470r
Connections:
- net GND: no longer CON1.4 (ID)
- net TX0: now also R4.1; no longer U1.25 (RXD)
- new net: R4.2, U1.25 (RXD)
- no-connect marks 44 -> 45
Other:
- note added: "Logo"
- note added: "Mounting Holes"
Changed lines of the file:
@@
 43 7C 02 00 00 84 0C F1 09 00 00 10 32 C4 27 00 00 40 C8 10 9F 00 00 00 21 43 7C 02 00 00 84 0C
 F1 09 00 00 10 32 C4 27 00 00 40 C8 10 9F 00 00 00 21 43 7C 02 00 00 84 EC FF 02 24 05 F2 19 03
-C8 1D 6B 00 00 00 00 49 45 4E 44 AE 42 60 82 01
+C8 1D 6B 00 00 00 00 49 45 4E 44 AE 42 60 82 00
 EndData
 $EndBitmap
@@
 Wire Wire Line
 	3050 6350 2350 6350
-Wire Wire Line
-	2350 6450 3050 6450
-Wire Wire Line
-	2350 6550 2350 6450
 $Comp
 L GND #PWR09
@@
 	1    0    0    -1
 $EndComp
-Wire Wire Line
-	2700 6500 2700 6450
-Connection ~ 2700 6450
 $Comp
 L C C7
@@
 P 6200 6250
 F 0 "R5" V 6280 6250 50  0000 C CNN
-F 1 "R" V 6207 6251 50  0000 C CNN
+F 1 "470r" V 6207 6251 50  0000 C CNN
 F 2 "" V 6130 6250 30  0000 C CNN
 F 3 "" H 6200 6250 30  0000 C CNN
@@
 $EndComp
 Wire Wire Line
-	5400 6150 5500 6150
+	5400 6150 5600 6150
 $Comp
 L C C8
@@
 Text Label 6450 6250 0    40   ~ 0
 RX0
-Text Label 5500 6150 0    40   ~ 0
+Text Label 6100 6150 0    40   ~ 0
 TX0
 Text Label 6850 6350 0    60   ~ 0
@@
 NoConn ~ 10200 4050
 NoConn ~ 10200 4550
+NoConn ~ 2350 6450
+Wire Wire Line
+	2350 6550 2600 6550
+Wire Wire Line
+	2600 6550 2600 6450
+Wire Wire Line
+	2600 6450 3050 6450
+Wire Wire Line
+	2700 6500 2700 6450
+Connection ~ 2700 6450
+Text Notes 10650 2400 0    60   ~ 0
+Logo
+Text Notes 10100 2700 0    60   ~ 0
+Mounting Holes
+$Comp
+L R R4
+U 1 1 579C49F3
+P 5850 6150
+F 0 "R4" V 5930 6150 50  0000 C CNN
+F 1 "470r" V 5857 6151 50  0000 C CNN
+F 2 "" V 5780 6150 30  0000 C CNN
+F 3 "" H 5850 6150 30  0000 C CNN
+	1    5850 6150
+	0    1    1    0
+$EndComp
 $EndSCHEMATC
