File: ATMega128_Breakout.kicad_pcb (KiCad board)
At the start: 2 copper layers, 25.4 x 53.3 mm, 21 parts, among them IC1 ATMEGA128-A, J2 SIL8, P1 CONN_10, P2 CONN_10, P3 CONN_10, P4 CONN_10, P5 CONN_01X01, P6 CONN_7, P8 CONN_5X2, SW1 rst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

Commit message: Updated Designs
Parts:
- removed C5: 0.1uF, Capacitors_SMD:C_0603_HandSoldering
- added C6: 0.1uF, Capacitors_SMD:C_0603_HandSoldering, B.Cu at (84.1, 55.6)
- added C7: 0.1uF, Capacitors_SMD:C_0603_HandSoldering, B.Cu at (84.1, 51.6)
- added C8: 0.1uF, Capacitors_SMD:C_0603_HandSoldering, B.Cu at (73.4, 55.9)
- added CON1: USB-MICRO-B, EE:USB_Micro-B_SMD_NEW, F.Cu at (78.7, 47.6)
- added P10: CONN_01X01, Connect:1pin, F.Cu at (89.5, 43.8)
- added P7: CONN_01X01, Connect:1pin, F.Cu at (67.9, 43.8)
- added P9: CONN_01X01, Connect:1pin, F.Cu at (89.5, 101.6)
- added R5: R, Resistors_SMD:R_0603_HandSoldering, B.Cu at (72.6, 52.3)
- added U1: CP2102, EE:cp2102_xl2, B.Cu at (78.7, 54.4)
- P6: value CONN_7 -> CONN_01X01; footprint Pin_Headers:Pin_Header_Straight_1x07 -> Connect:1pin
- moved J2 56.9 mm to (69.8, 98.6), turned to 90 degrees
- moved P8 42.1 mm to (83.8, 93.0), turned to 270 degrees
- moved P4 25.4 mm to (90.2, 69.8)
- moved P3 25.4 mm to (90.2, 72.4)
- moved X1 19.1 mm to (78.7, 61.0)
- moved C2 18.8 mm to (72.4, 61.0)
- moved C1 18.5 mm to (85.1, 61.0)
- moved P6 9.20 mm to (67.9, 101.6), turned to 0 degrees
- moved IC1 5.59 mm to (78.7, 73.7)
- moved P5 3.31 mm to (78.7, 53.3)
Connections:
- IC1 pad 62: /+5V -> /Aref
- J2 pad 1: /RX0 -> Net-(IC1-Pad35)
- J2 pad 2: /TX0 -> Net-(IC1-Pad36)
- J2 pad 3: Net-(IC1-Pad4) -> Net-(IC1-Pad37)
- J2 pad 4: Net-(IC1-Pad5) -> Net-(IC1-Pad38)
- J2 pad 5: Net-(IC1-Pad6) -> Net-(IC1-Pad39)
- J2 pad 6: Net-(IC1-Pad7) -> Net-(IC1-Pad40)
- J2 pad 7: Net-(IC1-Pad8) -> Net-(IC1-Pad41)
- J2 pad 8: Net-(IC1-Pad9) -> Net-(IC1-Pad42)
- P2 pad 1: Net-(P2-Pad1) -> /Aref
- P3 pad 1: /+5V -> /SCL
- P3 pad 2: GND -> /SDA
- P4 pad 1: Net-(IC1-Pad35) -> /RX0
- P4 pad 10: /SCL -> /+5V
- P4 pad 2: Net-(IC1-Pad36) -> /TX0
- P4 pad 3: Net-(IC1-Pad37) -> Net-(IC1-Pad4)
- P4 pad 4: Net-(IC1-Pad38) -> Net-(IC1-Pad5)
- P4 pad 5: Net-(IC1-Pad39) -> Net-(IC1-Pad6)
- P4 pad 6: Net-(IC1-Pad40) -> Net-(IC1-Pad7)
- P4 pad 7: Net-(IC1-Pad41) -> Net-(IC1-Pad8)
- P4 pad 8: Net-(IC1-Pad42) -> Net-(IC1-Pad9)
- P4 pad 9: /SDA -> GND
- P6 pad 1: GND -> Net-(P6-Pad1)
Other:
- board size 25.4 x 53.3 mm -> 25.4 x 61.6 mm
- board text added: "Aref"
- board text added: "ISP"
- board text added: "PB4"
- board text added: "PB5"
- board text added: "PC0"
- board text added: "PC1"
- board text added: "PC2"
- board text added: "PD5"
- board text added: "PD6"
- board text added: "PD7"
- board text added: "PF4"
- board text added: "PF5"
- board text added: "PF6"
- board text added: "PF7"
- board text removed: "2"
- board text removed: "4"
- board text removed: "5"
- board text removed: "5V"
- board text removed: "DTR"
- board text removed: "NC"
- board text removed: "PD0"
- board text removed: "PD1"
- board text removed: "PE0"
- board text removed: "PE1"
- board text removed: "PF0"
- board text removed: "PF1"
- board text removed: "R"
- board text removed: "T"

Commit message: Updated
Parts:
- added R4: 470r, Resistors_SMD:R_0603_HandSoldering, F.Cu at (82.8, 56.3)
- C1, C2, C3, C4, C6, C7, C8, R1, R2, R3, U1: moved to F.Cu
- P5: moved to B.Cu
- R5: value R -> 470r; moved to F.Cu
- moved C4 21.5 mm to (72.9, 85.1), turned to 0 degrees
- moved C3 21.0 mm to (83.7, 86.5), turned to 270 degrees
- moved C7 11.4 mm to (73.3, 55.4)
- moved C8 11.4 mm to (84.5, 53.1)
- moved R1 5.95 mm to (73.5, 88.1), turned to 90 degrees
- moved R5 2.80 mm to (74.8, 50.5)
- moved P5 2.16 mm to (78.6, 55.5), turned to 270 degrees
- moved C6 1.69 mm to (84.5, 57.3), turned to 270 degrees
- moved R2 0.51 mm to (71.6, 55.4)
- moved R3 0.38 mm to (86.1, 55.2)
- moved U1 0.28 mm to (78.6, 54.1)
- moved C2 0.25 mm to (72.1, 61.0), turned to 270 degrees
- moved C1 0.25 mm to (85.3, 61.0)
Connections:
- CON1 pad 4: GND -> Net-(CON1-Pad4)
- U1 pad 25: /TX0 -> Net-(R4-Pad2)
Other:
- board size 25.4 x 61.6 mm -> 25.4 x 62.9 mm
- board text added: "*"
- board text added: "+5V"
- board text added: "ExploreEmbedded.com"
- board text added: "PWM *"
- board text removed: "VCC"

Commit message: Routing
Parts:
- moved C8 17.0 mm to (71.0, 63.4), turned to 180 degrees
- moved C2 13.4 mm to (85.5, 60.0)
- moved C1 13.3 mm to (72.0, 60.0), turned to 270 degrees
- moved C4 12.2 mm to (84.9, 87.4), turned to 270 degrees
- moved C6 11.0 mm to (74.3, 53.1)
- moved R5 9.53 mm to (84.1, 52.5), turned to 270 degrees
- moved R2 2.41 mm to (71.3, 53.0)
- moved C7 2.28 mm to (72.8, 53.1)
- moved R3 2.22 mm to (85.9, 53.0)
- moved D1 1.71 mm to (71.3, 49.6)
- moved D3 1.64 mm to (85.9, 49.4)
- moved R4 1.41 mm to (84.1, 56.7), turned to 0 degrees
- moved C3 0.91 mm to (83.5, 87.4)
- moved CON1 0.28 mm to (78.7, 47.3)
- moved U1 0.14 mm to (78.7, 54.2)
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Routing:
- net GND: track 0.00 -> 181.5 mm, vias 0 -> 10
- net /+5V: track 0.00 -> 139.2 mm, vias 0 -> 11
- net /RX0: track 0.00 -> 89.9 mm, vias 0 -> 5
- net /TX0: track 0.00 -> 81.8 mm, vias 0 -> 3
- net /RST: track 0.00 -> 51.3 mm, vias 0 -> 3
- net /SCK: track 0.00 -> 47.9 mm, vias 0 -> 3
- net Net-(IC1-Pad60): track 0.00 -> 31.0 mm, vias 0 -> 2
- net /SDA: track 0.00 -> 30.8 mm, vias 0 -> 3
- net /SCL: track 0.00 -> 28.4 mm, vias 0 -> 3
- net Net-(C8-Pad1): track 0.00 -> 28.4 mm, vias 0 -> 4
- net Net-(IC1-Pad38): track 0.00 -> 28.1 mm, vias 0 -> 1
- net Net-(IC1-Pad57): track 0.00 -> 26.2 mm, vias 0 -> 2
- net Net-(IC1-Pad56): track 0.00 -> 25.9 mm, vias 0 -> 2
- net /Aref: track 0.00 -> 24.7 mm, vias 0 -> 1
- net Net-(IC1-Pad59): track 0.00 -> 24.1 mm, vias 0 -> 2
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- added copper zone on F.Cu, net /+5V
- added copper zone on B.Cu, net GND
Other:
- net class Default: clearance 0.1778 -> 0.1524
- rule trace_clearance: 0.1778 -> 0.1524
- rule via_min_drill: 0.508 -> 0.3
- rule via_min_size: 0.889 -> 0.6

Commit message: added name oneMicro to the board series
Other:
- board text added: "oneMicro"
- board text added: "oneMicro Atmega128"
